File: SPV1040.sch (KiCad schematic (older format))
At the start: 14 parts

Commit message: added current sensing circuit and 5v/3.3v voltage monitoring
Parts:
- U?: symbol CustomSymbols:SPV1040 -> Main-rescue:SPV1040-CustomSymbols
Changed lines of the file:
@@
 EESchema Schematic File Version 4
 LIBS:Main-cache
-LIBS:batteryCharger-cache
 EELAYER 29 0
 EELAYER END
 $Descr A4 11693 8268
 encoding utf-8
-Sheet 21 26
+Sheet 21 27
 Title ""
 Date ""
@@
 $EndComp
 $Comp
-L CustomSymbols:SPV1040 U?
+L Main-rescue:SPV1040-CustomSymbols U?
 U 1 1 5CCC8FA6
 P 5850 4150
@@
 AR Path="/5CC6D79E/5CCB70B2/5CCC8FA6" Ref="U?"  Part="1"
 AR Path="/5CC6D79E/5CCB7099/5CCC8FA6" Ref="U?"  Part="1"
+AR Path="/5CCC8FA6" Ref="U?"  Part="1"
 F 0 "U?" H 6000 5065 50  0000 C CNN
 F 1 "SPV1040" H 6000 4974 50  0000 C CNN
