File: BDR.sch (KiCad schematic (older format))
At the start: 9 parts

Commit message: added new timer circuit and changed deployment switch architecture
Connections:
- new net: R?.~, R?.~, U?.12 (FB)
Changed lines of the file:
@@
 $Descr A4 11693 8268
 encoding utf-8
-Sheet 34 35
+Sheet 34 34
 Title ""
 Date ""

Commit message: test commit
Connections:
- new net: R?.~, R?.~, U?.12 (FB)
Changed lines of the file:
@@
 $Descr A4 11693 8268
 encoding utf-8
-Sheet 34 34
+Sheet 34 33
 Title ""
 Date ""
